Commit message: wip(sim): Webots Phase 2.1 — replace inline Robot {} with PROTO (partial)
Replaces the inline Robot {} block in worlds_webots/mowgli_garden.wbt
with a local PROTO at protos/MowgliMower.proto, forked from the design
philosophy of Webots' shipped TurtleBot3Burger.proto and ROSbot.proto
(2 driving wheels + 1 caster ball on a BallJoint, wheels and caster
sharing the same z=0 ground-contact, narrow chassis bounding box well
clear of the floor).

**Status: PARTIAL.** This commit resolves the most egregious Phase 2
failure modes from commit ba57bc20 (chassis flips on its nose within
5 s, wheels never touching the floor) but still suffers from ~80–90 %
wheel-floor slip under cmd_vel, with the chassis settling at ~12°
forward pitch. Phase 1 forward-0.10-m/s reproduction:

  wheel-encoder integration: 0.49 m  (close to 0.50 m expected)
  GPS-grounded body motion:  0.05 m  (10 % of expected)
  chassis pitch at end:      ~12° forward

Phase 2 (sim_full_system.launch.py + COMMAND_START) was NOT exercised
because the slip leaves the robot too imprecise to reach Nav2 goals
within the FTC controller's tolerance.

What was tried (in order, none of which fixed the slip pathology):
  1. Front-caster TurtleBot3Burger-style (2 wheels + 1 caster behind).
     Robot tipped onto its rear in <5 s.
  2. Front caster instead of rear caster. Robot tipped forward.
  3. ROSbot-style joint dampingConstant=5 + staticFriction=1. No effect.
  4. Wheel boundingObject as Sphere (always-bottom contact) vs Cylinder.
     Marginal improvement.
  5. Wheel cylinder rotation aligned via inner Pose (Cylinder defaults
     to Z-axis in Webots; rotated -90° about X to align to body Y).
     Confirmed wheels touch the floor (was the original symptom — the
     un-rotated cylinder was a flat disc on its bottom face).
  6. HingeJoint axis flipped (0, 1, 0) → (0, -1, 0). Found the sign
     mismatch — with the natural axis, positive ω from
     diff_drive_controller drove the body BACKWARD (right-hand rule:
     +ω about +Y → wheel-bottom velocity in -X). Inverting matched the
     controller's convention.
  7. Chassis bounding box sizes from 0.40×0.30×0.16 down to
     0.10×0.10×0.05. Smaller helps a little but not enough.
  8. Chassis mass from 1 kg to 50 kg. Heavier reduces pitch but worsens
     translation.
  9. Motor maxTorque from 5 to 100 Nm. No effect.
 10. diff_drive_controller max_acceleration from 1.0 to 0.2 m/s². No effect.
 11. World coulombFriction from 0.8 to 5.0 to default. No effect.
 12. RotationalMotor consumptionFactor=-0.001 vs absent. No effect.
 13. COM positions: forward-of-axis (0.05, 0, 0.05), over-axis
     (0, 0, 0.05), low+forward (0.10, 0, 0.005). Shifts equilibrium
     pitch but slip ratio stays 80–90 %.
 14. Wheel mass from 0.1 to 4 kg. Heavier wheels → worse pitch + the
     robot drives BACKWARD (chassis flips past 90°).

Final settled values (best honest attempt — robot drives forward
at ~10 % efficiency, stable pitch ~12°):
  * wheels at body x=0, y=±0.1625, z=0.093, mass 0.5 kg, axis (0,-1,0)
  * caster at body (+0.20, 0, 0.04), sphere radius 0.04
  * chassis bbox 0.30×0.28×0.08 m at z=0.25 (well clear of floor)
  * total mass 8.76 kg, COM at (0, 0, 0.05)
  * dampingConstant=5, staticFriction=1, maxTorque=100, maxVelocity=21.5
  * world ContactProperties: Webots defaults (no override)

Likely next investigations:
  * Webots' wheel-floor contact model with softCFM/softERP tuning.
  * Why diff_drive_controller's reported wheel ω matches setpoint
    while body motion is ~10 % of expected — possible velocity
    clamping at the hardware-interface boundary.
  * PROTO with kinematic TRUE wheels (skip ODE physics for the
    drive train).
  * 4-wheel layout (no caster) following ROSbot's exact PROTO,
    scaled to Mowgli geometry.
  * Adopt webots_ros2_husarion's RosbotXL as a starting point.

Other companion changes:
  * urdf_webots/mowgli_webots.urdf: wheel joint origin z = -0.007
    (was -0.10 — wheels were buried in the floor). Effort 20 (was 10)
    to match the new motor maxTorque headroom.
  * CMakeLists.txt: install protos/ directory.
  * worlds_webots/mowgli_garden.wbt: instantiate the PROTO,
    sensors via extensionSlot, drop the custom contactProperties
    (Webots default behaviour was identical).

File: ros2/src/mowgli_simulation/urdf_webots/mowgli_webots.urdf (robot description, URDF)
Before this commit: robot MowgliMower, 7 links, 6 joints
Joints:
- joint left_wheel_motor: limit effort=10.0 velocity=100.0 -> effort=20.0 velocity=100.0; origin xyz=0 0.1625 -0.10 rpy=0 0 0 -> xyz=0 0.1625 -0.007 rpy=0 0 0
- joint right_wheel_motor: limit effort=10.0 velocity=100.0 -> effort=20.0 velocity=100.0; origin xyz=0 -0.1625 -0.10 rpy=0 0 0 -> xyz=0 -0.1625 -0.007 rpy=0 0 0

Commit message: fix(sim): YardForce 500 chassis dimensions in Webots PROTO + URDF
Phase 2.1 PROTO had a placeholder chassis (0.30x0.30x0.10 m, 1 caster)
that did not match the YardForce 500 hardware. Operator flagged
'robot shape is wrong' on Foxglove inspection.

Now matches the real YardForce 500 + mowgli_robot.yaml:
  * Chassis 0.60x0.40x0.19 m, mass 8.76 kg
  * Centred at chassis_center_x = +0.18 m forward of base_link
  * Two motorised rear wheels at base_link, track 0.325, radius 0.093
  * Two passive front casters at +0.30 m forward, track 0.36

URDF static TF aligned:
  * base_footprint to base_link: z=0.093 (= wheel_radius)
  * lidar_link: xyz='0 0.024 0.290' (centred, +10cm above chassis top)
  * imu_link: xyz='0.18 0 0.095' (chassis centre per yaml)
  * gps_link: xyz='0.30 0 0.190' (front-top per yaml)

.wbt extensionSlot sensor positions updated to land sensors at the
URDF static TF positions in world coords.

KinematicDrive bypasses physics so this is a visual/TF/footprint
correctness fix; trajectory chaos #200 is unchanged.

File: ros2/src/mowgli_simulation/urdf_webots/mowgli_webots.urdf (robot description, URDF)
Before this commit: robot MowgliMower, 7 links, 6 joints
Joints:
- joint base_footprint_to_base_link: origin xyz=0 0 0.10 rpy=0 0 0 -> xyz=0 0 0.093 rpy=0 0 0
- joint base_link_to_gps: origin xyz=0.30 0 0.10 rpy=0 0 0 -> xyz=0.30 0 0.19 rpy=0 0 0
- joint base_link_to_imu: origin xyz=0 0 0 rpy=0 0 0 -> xyz=0.18 0 0.095 rpy=0 0 0
- joint base_link_to_lidar: origin xyz=0 0.024 0.12 rpy=0 0 3.1408 -> xyz=0 0.024 0.290 rpy=0 0 3.1408
- joint left_wheel_motor: origin xyz=0 0.1625 -0.007 rpy=0 0 0 -> xyz=0 0.1625 0 rpy=0 0 0
- joint right_wheel_motor: origin xyz=0 -0.1625 -0.007 rpy=0 0 0 -> xyz=0 -0.1625 0 rpy=0 0 0
