Commit message: refactor(mowgli_hardware): migrate drive base to ros2_control
Replace the hand-rolled host wheel-velocity PI + gyro angular-rate loop
with the standard ros2_control stack: diff_drive_controller -> chained
pid_controller x2 -> MowgliSystemInterface, a hardware_interface plugin
that owns the STM32 COBS serial link and embeds the HardwareBridgeNode
comms core.

Why: the gyro angular-rate loop oscillated on tight U-turns (the FTC
limit-cycle, gyro +-2.0 rad/s on a +-0.8 cmd). It is removed by design —
the per-wheel velocity loop (stock pid_controller) absorbs the nonlinear
PWM curve and the localizer owns heading. The plugin only inverts the
firmware deadband (velocity_pwm.hpp) to raw PWM and relays it.

The comms core keeps ALL non-motor I/O verbatim (IMU+cal, status/power/
battery, blade, emergency+heartbeat, HL-state, charging, dock-heading,
/wheel_odom with force-zero-on-charging + non-holo covariances). There is
no standalone hardware_bridge_node executable — controller_manager owns
the serial link. diff_drive_controller.enable_odom_tf=false (fusion_graph
owns odom->base_footprint); wheel_radius/separation are injected from the
same mowgli_robot.yaml the plugin uses so they cannot diverge.

Deletes wheel_rate_controller.hpp, angular_rate_controller.hpp, their
tests, and the now-dead hardware_bridge.yaml. mowgli_hardware builds
clean locally; 108 tests pass.

On-robot pivot-accuracy validation (gyro loop removed) is deferred — the
robot must not move during the migration.

File: ros2/src/mowgli_bringup/urdf/mowgli.urdf.xacro (robot description, xacro)
@@ -53,4 +53,22 @@
   <xacro:arg name="caster_track"     default="0.36"/>
   <xacro:arg name="blade_radius"     default="0.09"/>
+  <!-- ros2_control hardware interface (real STM32 drive base). The motor path
+       is diff_drive_controller → pid_controller ×2 → MowgliSystemInterface,
+       which owns the COBS serial link. These args are injected by the launch
+       from mowgli_robot.yaml. use_ros2_control:=false drops the block (e.g.
+       when only TF/visualisation is wanted). -->
+  <xacro:arg name="use_ros2_control"     default="true"/>
+  <xacro:arg name="serial_port"          default="/dev/mowgli"/>
+  <xacro:arg name="baud_rate"            default="115200"/>
+  <xacro:arg name="ticks_per_meter"      default="220.0"/>
+  <xacro:arg name="wheel_meas_filter_tau" default="0.12"/>
+  <xacro:arg name="pwm_per_mps"          default="300.0"/>
+  <xacro:arg name="deadband_pwm"         default="40.0"/>
+  <xacro:arg name="max_pwm"              default="255.0"/>
+  <xacro:arg name="dock_pose_x"          default="0.0"/>
+  <xacro:arg name="dock_pose_y"          default="0.0"/>
+  <xacro:arg name="dock_pose_yaw"        default="0.0"/>
+  <xacro:arg name="imu_cal_samples"      default="1000"/>
+  <xacro:arg name="lift_recovery_mode"   default="false"/>
   <!-- ================================================================
        Properties (resolved from args — all shape from config)
@@ -364,4 +382,43 @@
   </joint>
   <!-- ================================================================
+       ros2_control hardware interface (real STM32 drive base)
+       ================================================================ -->
+  <xacro:if value="$(arg use_ros2_control)">
+    <ros2_control name="MowgliDriveBase" type="system">
+      <hardware>
+        <plugin>mowgli_hardware/MowgliSystemInterface</plugin>
+        <!-- Serial link -->
+        <param name="serial_port">$(arg serial_port)</param>
+        <param name="baud_rate">$(arg baud_rate)</param>
+        <param name="serial_rx_timeout_s">2.0</param>
+        <!-- Tick→metre scale (sole ground scale) + joint-angle conversion -->
+        <param name="ticks_per_meter">$(arg ticks_per_meter)</param>
+        <param name="wheel_radius">$(arg wheel_radius)</param>
+        <param name="wheel_track">$(arg wheel_track)</param>
+        <param name="wheel_meas_filter_tau">$(arg wheel_meas_filter_tau)</param>
+        <!-- velocity (m/s) → PWM feedforward (inverts the firmware deadband) -->
+        <param name="pwm_per_mps">$(arg pwm_per_mps)</param>
+        <param name="deadband_pwm">$(arg deadband_pwm)</param>
+        <param name="max_pwm">$(arg max_pwm)</param>
+        <!-- Comms-core node params (dock pose, IMU calibration) -->
+        <param name="dock_pose_x">$(arg dock_pose_x)</param>
+        <param name="dock_pose_y">$(arg dock_pose_y)</param>
+        <param name="dock_pose_yaw">$(arg dock_pose_yaw)</param>
+        <param name="imu_cal_samples">$(arg imu_cal_samples)</param>
+        <param name="lift_recovery_mode">$(arg lift_recovery_mode)</param>
+      </hardware>
+      <joint name="left_wheel_joint">
+        <command_interface name="velocity"/>
+        <state_interface name="position"/>
+        <state_interface name="velocity"/>
+      </joint>
+      <joint name="right_wheel_joint">
+        <command_interface name="velocity"/>
+        <state_interface name="position"/>
+        <state_interface name="velocity"/>
+      </joint>
+    </ros2_control>
+  </xacro:if>
+  <!-- ================================================================
        Gazebo simulation
        ================================================================ -->
