Commit message: feat(gui): render layered mower assemblies and matching dock

File: ros2/src/mowgli_bringup/urdf/mowgli.urdf.xacro (robot description, xacro)
@@ -70,4 +70,6 @@
   <xacro:arg name="caster_radius"    default="0.03"/>
   <xacro:arg name="caster_track"     default="0.36"/>
+  <!-- -1 preserves the historical chassis-derived caster axle position. -->
+  <xacro:arg name="caster_x_offset"  default="-1.0"/>
   <xacro:arg name="blade_radius"     default="0.09"/>
   <!-- ================================================================
@@ -87,5 +89,6 @@
   <xacro:property name="caster_mass"      value="0.2"/>
   <!-- Casters near front edge of chassis -->
-  <xacro:property name="caster_x_offset"  value="${chassis_cx + base_length/2.0 - caster_radius}"/>
+  <xacro:property name="configured_caster_x" value="$(arg caster_x_offset)"/>
+  <xacro:property name="caster_x_offset" value="${chassis_cx + base_length/2.0 - caster_radius if float(configured_caster_x) == -1.0 else float(configured_caster_x)}"/>
   <xacro:property name="caster_track"     value="$(arg caster_track)"/>
   <xacro:property name="base_mass"        value="$(arg chassis_mass_kg)"/>

Commit message: feat(gui): add configurable chassis vertical placement

File: ros2/src/mowgli_bringup/urdf/mowgli.urdf.xacro (robot description, xacro)
@@ -58,4 +58,6 @@
   <xacro:arg name="chassis_width"    default="0.40"/>
   <xacro:arg name="chassis_height"   default="0.19"/>
+  <!-- Shell bottom relative to axle; photo-estimated YardForce default. -->
+  <xacro:arg name="chassis_z_offset" default="-0.05"/>
   <xacro:arg name="chassis_mass_kg"  default="8.76"/>
   <xacro:arg name="chassis_center_x" default="0.20"/>
@@ -79,4 +81,5 @@
   <xacro:property name="base_width"       value="$(arg chassis_width)"/>
   <xacro:property name="base_height"      value="$(arg chassis_height)"/>
+  <xacro:property name="chassis_z_offset" value="$(arg chassis_z_offset)"/>
   <xacro:property name="chassis_cx"       value="$(arg chassis_center_x)"/>
   <xacro:property name="wheel_radius"     value="$(arg wheel_radius)"/>
@@ -153,5 +156,5 @@
     <visual>
       <!-- Chassis centre offset forward from wheel axis -->
-      <origin xyz="${chassis_cx} 0 ${base_height/2}" rpy="0 0 0"/>
+      <origin xyz="${chassis_cx} 0 ${base_height/2 + chassis_z_offset}" rpy="0 0 0"/>
       <geometry>
         <box size="${base_length} ${base_width} ${base_height}"/>
@@ -162,5 +165,5 @@
     </visual>
     <collision>
-      <origin xyz="${chassis_cx} 0 ${base_height/2}" rpy="0 0 0"/>
+      <origin xyz="${chassis_cx} 0 ${base_height/2 + chassis_z_offset}" rpy="0 0 0"/>
       <geometry>
         <box size="${base_length} ${base_width} ${base_height}"/>
